Commit message: Finished the robot urdf model

File: urdf/bilkins.urdf (robot description, URDF)
Before this commit: robot Bilkins, 5 links, 4 joints
Joints:
- joint front_axle_to_chassis: origin xyz=-1.3 0 0.5 rpy=0 0 0 -> xyz=-1.3 0 0.5
- joint front_left_wheel_to_axle: axis (none) -> 0 1 0; origin (none) -> xyz=0 -0.9 0; type fixed -> continuous
- joint front_right_wheel_to_axle: axis (none) -> 0 1 0; origin (none) -> xyz=0 0.9 0; type fixed -> continuous

Commit message: Added collision elements to the model

File: urdf/bilkins.urdf (robot description, URDF)
Before this commit: robot Bilkins, 5 links, 4 joints
Links:
- link base_link: geometry collision mesh filename=package://bilkins/meshes/chassis.dae scale=0.1 0.1 0.1; visual mesh filename=package://bilkins/meshes/chassis.dae scale=0.1 0.1 0.1
- link front_axle: geometry collision mesh filename=package://bilkins/meshes/front_axle.dae scale=0.1 0.1 0.1; visual mesh filename=package://bilkins/meshes/front_axle.dae scale=0.1 0.1 0.1
- link front_left_wheel: geometry collision mesh filename=package://bilkins/meshes/front_left_wheel.dae scale=0.1 0.1 0.1; visual mesh filename=package://bilkins/meshes/front_left_wheel.dae scale=0.1 0.1 0.1
- link front_right_wheel: geometry collision mesh filename=package://bilkins/meshes/front_right_wheel.dae scale=0.1 0.1 0.1; visual mesh filename=package://bilkins/meshes/front_right_wheel.dae scale=0.1 0.1 0.1
- link rear_axle: geometry collision mesh filename=package://bilkins/meshes/rear_axle.dae scale=0.1 0.1 0.1; visual mesh filename=package://bilkins/meshes/rear_axle.dae scale=0.1 0.1 0.1

Commit message: Added a launch file for loading the robot up in Gazebo

File: urdf/bilkins.urdf (robot description, URDF)
Before this commit: robot Bilkins, 5 links, 4 joints
Links:
- removed link base_link
- added link chassis, mass 0.2; collision mesh filename=package://bilkins/meshes/chassis.dae scale=0.1 0.1 0.1; visual mesh filename=package://bilkins/meshes/chassis.dae scale=0.1 0.1 0.1
- added link hokuyo_link, mass 1e-5; collision box size=1 1 1; visual mesh filename=package://bilkins/meshes/hokuyo.dae
Joints:
- added joint hokuyo_joint: type fixed, parent chassis, child hokuyo_link, origin xyz=0 0 0 rpy=0 0 0, axis 0 1 0
- joint front_axle_to_chassis: parent base_link -> chassis
- joint rear_axle_to_chassis: parent base_link -> chassis

Commit message: Added the hokuyo laser scanner to the model and placed it in the correct location

File: urdf/bilkins.urdf (robot description, URDF)
Before this commit: robot Bilkins, 6 links, 5 joints
Links:
- link hokuyo_link: geometry collision box size=0.1 0.1 0.1; visual mesh filename=package://bilkins/meshes/hokuyo.dae

Commit message: Added actuators to the urdf file and several additional files that regard the odometry and navigation of the robot

File: urdf/bilkins.urdf (robot description, URDF)
Before this commit: robot Bilkins, 6 links, 5 joints
Links:
- removed link chassis
- added link base_link, mass 0.2; collision mesh filename=package://bilkins/meshes/chassis.dae scale=0.1 0.1 0.1; visual mesh filename=package://bilkins/meshes/chassis.dae scale=0.1 0.1 0.1
- added link camera_link, mass 1e-5; collision box size=0.1 0.1 0.1; visual box size=0.1 0.1 0.1
Joints:
- added joint camera_joint: type fixed, parent base_link, child camera_link, origin xyz=-1.1 0 0.7 rpy=3.14 3.14 3.14, axis 0 1 0
- joint front_axle_to_chassis: parent chassis -> base_link
- joint hokuyo_joint: origin xyz=0 0 0 rpy=0 0 0 -> xyz=-1 0 1.2 rpy=3.14 3.14 0; parent chassis -> base_link
- joint rear_axle_to_chassis: parent chassis -> base_link
